File: pcb/crossingsignals.sch (EAGLE design)
At the start: 33 parts, among them J1 DETECT_4_SEND, J11 DEBUG, J2 DETECT_4_RCV, J3 DETECT_3_SEND, J4 DETECT_3_RCV, J5 DETECT_2_SEND, J6 DETECT_2_RCV, J7 DETECT_1_SEND, J8 DETECT_1_RCV, J9 POWER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

Commit message: Adding a semaphore
* Add a GPIO signal to act as a semaphore in case anyone wants to know
when the signals are turned on or off
* Fix the handling of the interrupts. It's not individual functions and
should be smarter
Parts:
- added J10: SIGNAL, SparkFun-Connectors:CONN_02
Connections:
- new net GP17: J10.1, X1.GP17
- net GND: now also J10.2
Changed lines of the file:
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@@
 <part name="D1" library="adafruit" library_urn="urn:adsk.eagle:library:420" deviceset="1N4004" device="" package3d_urn="urn:adsk.eagle:package:6240344/1"/>
 <part name="C1" library="SparkFun-Capacitors" library_urn="urn:adsk.eagle:library:510" deviceset="100UF-POLAR" device="-RADIAL-2.5MM-25V-20%" package3d_urn="urn:adsk.eagle:package:37415/1" value="100uF"/>
+<part name="J10" library="SparkFun-Connectors" library_urn="urn:adsk.eagle:library:513" deviceset="CONN_02" device="" package3d_urn="urn:adsk.eagle:package:38039/1" value="SIGNAL"/>
 </parts>
 <sheets>
@@
 <attribute name="VALUE" x="191.516" y="77.089" size="1.778" layer="96" font="vector"/>
 </instance>
+<instance part="J10" gate="G$1" x="20.32" y="109.22" smashed="yes">
+<attribute name="VALUE" x="17.78" y="104.394" size="1.778" layer="96" font="vector"/>
+<attribute name="NAME" x="17.78" y="114.808" size="1.778" layer="95" font="vector"/>
+</instance>
 </instances>
 <busses>
@@
 <junction x="190.5" y="76.2"/>
 <label x="180.34" y="76.2" size="1.016" layer="95" rot="R180" xref="yes"/>
+</segment>
+<segment>
+<pinref part="J10" gate="G$1" pin="2"/>
+<wire x1="27.94" y1="111.76" x2="43.18" y2="111.76" width="0.1524" layer="91"/>
+<label x="43.18" y="111.76" size="1.016" layer="95" xref="yes"/>
 </segment>
 </net>
@@
 </segment>
 </net>
+<net name="GP17" class="0">
+<segment>
+<pinref part="J10" gate="G$1" pin="1"/>
+<wire x1="27.94" y1="109.22" x2="43.18" y2="109.22" width="0.1524" layer="91"/>
+<label x="43.18" y="109.22" size="1.016" layer="95" xref="yes"/>
+</segment>
+<segment>
+<pinref part="X1" gate="G$1" pin="GP17"/>
+<wire x1="162.56" y1="152.4" x2="175.26" y2="152.4" width="0.1524" layer="91"/>
+<label x="175.26" y="152.4" size="1.016" layer="95" xref="yes"/>
+</segment>
+</net>
